File: kicad/data.sch (KiCad schematic (older format))
At the start: 46 parts, among them IC2 Si8663AB-B-IS1, IC3 MAX3387ECUG+, IC4 VOR1121B6T, J2 USB_C, J3 XCVR_CAT_TTL, J4 FTDI header, J5 PTT choice, J6 XCVR_PTT, J7 XCVR_CAT_RS232, U1 SN65220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

Commit message: Change DC-DC convertor; other small changes
* Change RFM-0505S (unregulated) to PQS075-S5-S5-S (regulated)
* Naming conventions
* Alignment
Parts:
- renumbered U1 to U3, IC2 to U4, U2 to U5, IC3 to U6, IC4 to U7
Changed lines of the file:
@@
 P 1750 3200
 AR Path="/5FABC8C9" Ref="U?"  Part="1"
-AR Path="/5F9E7705/5FABC8C9" Ref="U1"  Part="1"
-F 0 "U1" H 1750 3425 50  0000 C CNN
+AR Path="/5F9E7705/5FABC8C9" Ref="U3"  Part="1"
+F 0 "U3" H 1750 3425 50  0000 C CNN
 F 1 "SN65220" H 1750 3334 50  0000 C CNN
 F 2 "Package_TO_SOT_SMD:SOT-23-6" H 2100 3050 50  0001 L CNN
@@
 P 4550 2650
 AR Path="/5FADB66C" Ref="U?"  Part="1"
-AR Path="/5F9E7705/5FADB66C" Ref="U2"  Part="1"
-F 0 "U2" H 4550 2650 50  0000 C CNN
+AR Path="/5F9E7705/5FADB66C" Ref="U5"  Part="1"
+F 0 "U5" H 4550 2650 50  0000 C CNN
 F 1 "FT232RL" H 4550 2550 50  0000 C CNN
 F 2 "Package_SO:SSOP-28_5.3x10.2mm_P0.65mm" H 5650 1750 50  0001 C CNN
@@
 Power
 $Comp
-L custom:MAX3387ECUG+ IC3
+L custom:MAX3387ECUG+ U6
 U 1 1 60048EC4
 P 8400 3300
-F 0 "IC3" H 9150 2800 50  0000 C CNN
+F 0 "U6" H 9150 2800 50  0000 C CNN
 F 1 "MAX3387ECUG+" H 9150 2700 50  0000 C CNN
 F 2 "SOP65P640X110-24N" H 11800 3300 50  0001 L CNN
@@
 XCVR_GND
 $Comp
-L custom:Si8663AB-B-IS1 IC2
+L custom:Si8663AB-B-IS1 U4
 U 1 1 60364EF5
 P 2400 6100
-F 0 "IC2" H 3000 6450 50  0000 C CNN
+F 0 "U4" H 3000 6450 50  0000 C CNN
 F 1 "Si8663AB-B-IS1" H 3000 5700 50  0000 C CNN
 F 2 "SOIC127P600X175-16N" H 4400 6200 50  0001 L CNN
@@
 Isolation
 $Comp
-L custom:VOR1121B6T IC4
+L custom:VOR1121B6T U7
 U 1 1 5F9F5535
 P 8950 1200
-F 0 "IC4" H 9400 1465 50  0000 C CNN
+F 0 "U7" H 9400 1465 50  0000 C CNN
 F 1 "VOR1121B6T" H 9400 1374 50  0000 C CNN
 F 2 "SOT254P980X380-6N" H 10300 1300 50  0001 L CNN
