File: kicad/power.sch (KiCad schematic (older format))
At the start: 9 parts, among them IC1 L78M05CDT-TR, J1 XCVR power choice

Commit message: Change DC-DC convertor; other small changes
* Change RFM-0505S (unregulated) to PQS075-S5-S5-S (regulated)
* Naming conventions
* Alignment
Parts:
- removed PS1: RFM-0505S, RFM0505S, symbol custom:RFM-0505S
- added U1: PQS075-S5-S5-S, symbol custom:PQS075-S5-S5-S
- C1: value 10u -> 4.7u
- C2: value 330p -> 4.7u
- C3: value 330p -> 10u
- L1: value 22u -> 6.8u
- renumbered IC1 to U2
Connections:
- wire segments 36 -> 32
Other:
- note added: "* Isolated 5V power supply for RS232 driver and optocoupler\n* See datasheet p6 for EMC filtration"
- note removed: "* Isolated 5V power supply for RS232 driver and optocoupler\n* See datasheet p3 for EMC filtration\n* 330pF caps rated for 1kV"
- moved on the sheet: C4, C5, U2
Changed lines of the file:
@@
 Comment4 ""
 $EndDescr
-Text Notes 3000 4750 0    39   ~ 0
-* Isolated 5V power supply for RS232 driver and optocoupler\n* See datasheet p3 for EMC filtration\n* 330pF caps rated for 1kV
-Text Notes 6650 4100 0    39   ~ 0
-* Regulated 5V power supply for RS232 driver and optocoupler\n* See Fig. 4 of datasheet
+Text Notes 3250 4400 0    39   ~ 0
+* Isolated 5V power supply for RS232 driver and optocoupler\n* See datasheet p6 for EMC filtration
 $Comp
 L Connector_Generic:Conn_01x03 J?
@@
 Text Notes 5800 2800 2    39   ~ 0
 One jumper
-Text GLabel 7200 3000 0    50   Input ~ 0
-XCVR_GND
-Wire Wire Line
-	7300 3200 7300 3100
-Wire Wire Line
-	7300 3000 7200 3000
-Wire Wire Line
-	8000 3100 7300 3100
-Connection ~ 7300 3100
-Wire Wire Line
-	7300 3100 7300 3000
-Wire Wire Line
-	6600 3100 7300 3100
-$Comp
-L custom:RFM-0505S PS1
-U 1 1 60911470
-P 3450 3600
-F 0 "PS1" H 3800 3150 50  0000 C CNN
-F 1 "RFM-0505S" H 3950 3450 50  0000 C CNN
-F 2 "RFM0505S" H 5450 3700 50  0001 L CNN
-F 3 "https://www.recom-power.com/pdf/Econoline/RFM.pdf" H 5450 3600 50  0001 L CNN
-F 4 "RECOM POWER - RFM-0505S - DC-DC CONVERTER, 5V, 0.2A" H 5450 3500 50  0001 L CNN "Description"
-F 5 "10.5" H 5450 3400 50  0001 L CNN "Height"
-F 6 "919-RFM-0505S" H 5450 3300 50  0001 L CNN "Mouser Part Number"
-F 7 "https://www.mouser.co.uk/ProductDetail/RECOM-Power/RFM-0505S?qs=lYGu3FyN48dRVYKTH5ipqg%3D%3D" H 5450 3200 50  0001 L CNN "Mouser Price/Stock"
-F 8 "RECOM Power" H 5450 3100 50  0001 L CNN "Manufacturer_Name"
-F 9 "RFM-0505S" H 5450 3000 50  0001 L CNN "Manufacturer_Part_Number"
-	1    3450 3600
-	1    0    0    -1
-$EndComp
-Wire Wire Line
-	6600 3250 6600 3100
-Connection ~ 6600 3600
-Wire Wire Line
-	6600 3450 6600 3600
-$Comp
-L Device:C_Small C?
-U 1 1 608AF3CD
-P 6600 3350
-AR Path="/608AF3CD" Ref="C?"  Part="1"
-AR Path="/5F9D7A3C/608AF3CD" Ref="C4"  Part="1"
-F 0 "C4" H 6692 3396 50  0000 L CNN
-F 1 "100n" H 6692 3305 50  0000 L CNN
-F 2 "" H 6600 3350 50  0001 C CNN
-F 3 "~" H 6600 3350 50  0001 C CNN
-	1    6600 3350
-	-1   0    0    1
-$EndComp
-Wire Wire Line
-	8000 3250 8000 3100
-Wire Wire Line
-	8000 3600 7900 3600
-Connection ~ 8000 3600
-Wire Wire Line
-	8000 3450 8000 3600
-$Comp
-L Device:C_Small C?
-U 1 1 608AC7D8
-P 8000 3350
-AR Path="/608AC7D8" Ref="C?"  Part="1"
-AR Path="/5F9D7A3C/608AC7D8" Ref="C5"  Part="1"
-F 0 "C5" H 8092 3396 50  0000 L CNN
-F 1 "330n" H 8092 3305 50  0000 L CNN
-F 2 "" H 8000 3350 50  0001 C CNN
-F 3 "~" H 8000 3350 50  0001 C CNN
-	1    8000 3350
-	1    0    0    -1
-$EndComp
-Wire Wire Line
-	6700 3600 6600 3600
-Wire Wire Line
-	8100 3600 8000 3600
-Text GLabel 8100 3600 2    50   Input ~ 0
-XCVR_VCC
-$Comp
-L custom:L78M05CDT-TR IC1
-U 1 1 608A3B2A
-P 7900 3600
-F 0 "IC1" H 8500 3865 50  0000 C CNN
-F 1 "L78M05CDT-TR" H 8500 3774 50  0000 C CNN
-F 2 "L78M05CDTTR" H 10450 3850 50  0001 L CNN
-F 3 "https://componentsearchengine.com/Datasheets/2/L78M05CDT-TR.pdf" H 10450 3750 50  0001 L CNN
-F 4 "Linear Voltage Regulators 5.0V 0.5A Positive" H 10450 3650 50  0001 L CNN "Description"
-F 5 "2.4" H 10450 3550 50  0001 L CNN "Height"
-F 6 "511-L78M05CDT-TR" H 10450 3450 50  0001 L CNN "Mouser Part Number"
-F 7 "https://www.mouser.co.uk/ProductDetail/STMicroelectronics/L78M05CDT-TR?qs=JIXmGdi%252BcuKa7ml6d%2FqNIw%3D%3D" H 10450 3350 50  0001 L CNN "Mouser Price/Stock"
-F 8 "STMicroelectronics" H 10450 3250 50  0001 L CNN "Manufacturer_Name"
-F 9 "L78M05CDT-TR" H 10450 3150 50  0001 L CNN "Manufacturer_Part_Number"
-	1    7900 3600
-	-1   0    0    1
-$EndComp
-Text Notes 3950 2900 1    50   ~ 0
+Text Notes 3950 3000 1    50   ~ 0
 Isolation
 $Comp
@@
 AR Path="/5F9D7A3C/60943CCC" Ref="L1"  Part="1"
 F 0 "L1" V 3050 3600 50  0000 C CNN
-F 1 "22u" V 3150 3600 50  0000 C CNN
+F 1 "6.8u" V 3150 3600 50  0000 C CNN
 F 2 "" H 3100 3600 50  0001 C CNN
 F 3 "~" H 3100 3600 50  0001 C CNN
@@
 Wire Wire Line
 	2750 3600 2900 3600
-Wire Wire Line
-	3200 3600 3400 3600
 $Comp
 L power:GND #PWR?
@@
 AR Path="/60949AAC" Ref="C?"  Part="1"
 AR Path="/5F9D7A3C/60949AAC" Ref="C1"  Part="1"
-F 0 "C1" H 2950 3700 50  0000 C CNN
-F 1 "10u" H 2800 3800 50  0000 C CNN
+F 0 "C1" H 3000 3700 50  0000 C CNN
+F 1 "4.7u" H 3000 3800 50  0000 C CNN
 F 2 "" H 2900 3750 50  0001 C CNN
 F 3 "~" H 2900 3750 50  0001 C CNN
@@
 	2900 3850 2900 3900
 Connection ~ 2900 3900
-Wire Wire Line
-	2900 3900 3400 3900
-Wire Wire Line
-	4450 3600 4500 3600
-Wire Wire Line
-	4450 3900 4500 3900
-$Comp
-L Device:C_Small C?
-U 1 1 6094E417
-P 3950 3250
-AR Path="/6094E417" Ref="C?"  Part="1"
-AR Path="/5F9D7A3C/6094E417" Ref="C2"  Part="1"
-F 0 "C2" V 3850 3100 50  0000 L CNN
-F 1 "330p" V 4050 3050 50  0000 L CNN
-F 2 "" H 3950 3250 50  0001 C CNN
-F 3 "~" H 3950 3250 50  0001 C CNN
-	1    3950 3250
-	0    1    1    0
-$EndComp
-Wire Wire Line
-	3400 3600 3400 3250
-Wire Wire Line
-	3400 3250 3850 3250
-Connection ~ 3400 3600
-Wire Wire Line
-	3400 3600 3450 3600
-Wire Wire Line
-	4050 3250 4500 3250
-Wire Wire Line
-	4500 3250 4500 3600
-Connection ~ 4500 3600
-$Comp
-L Device:C_Small C?
-U 1 1 609519C5
-P 3950 4350
-AR Path="/609519C5" Ref="C?"  Part="1"
-AR Path="/5F9D7A3C/609519C5" Ref="C3"  Part="1"
-F 0 "C3" V 3850 4200 50  0000 L CNN
-F 1 "330p" V 4050 4150 50  0000 L CNN
-F 2 "" H 3950 4350 50  0001 C CNN
-F 3 "~" H 3950 4350 50  0001 C CNN
-	1    3950 4350
-	0    1    1    0
-$EndComp
-Wire Wire Line
-	3400 3900 3400 4350
-Wire Wire Line
-	3400 4350 3850 4350
-Connection ~ 3400 3900
-Wire Wire Line
-	3400 3900 3450 3900
-Wire Wire Line
-	4050 4350 4500 4350
-Wire Wire Line
-	4500 4350 4500 3900
-Connection ~ 4500 3900
-Wire Wire Line
-	4500 3900 4900 3900
 Wire Notes Line
-	3950 4100 3950 2550
+	3950 4200 3950 2650
 Text GLabel 4900 3900 2    50   Input ~ 0
 XCVR_GND
@@
 	5550 3600 5550 3250
 Wire Wire Line
-	4500 3600 5550 3600
-Wire Wire Line
 	5750 3600 5750 3250
+Text Notes 6550 4450 0    39   ~ 0
+* Regulated 5V power supply for RS232 driver and optocoupler\n* See Fig. 4 of datasheet
+Text GLabel 7200 4200 0    50   Input ~ 0
+XCVR_GND
+Wire Wire Line
+	7300 4000 7300 4100
+Wire Wire Line
+	7300 4200 7200 4200
+Wire Wire Line
+	8000 4100 7300 4100
+Connection ~ 7300 4100
+Wire Wire Line
+	7300 4100 7300 4200
+Wire Wire Line
+	6600 4100 7300 4100
+Wire Wire Line
+	6600 3950 6600 4100
+Connection ~ 6600 3600
+Wire Wire Line
+	6600 3750 6600 3600
+$Comp
+L Device:C_Small C?
+U 1 1 608AF3CD
+P 6600 3850
+AR Path="/608AF3CD" Ref="C?"  Part="1"
+AR Path="/5F9D7A3C/608AF3CD" Ref="C4"  Part="1"
+F 0 "C4" H 6692 3896 50  0000 L CNN
+F 1 "100n" H 6692 3805 50  0000 L CNN
+F 2 "" H 6600 3850 50  0001 C CNN
+F 3 "~" H 6600 3850 50  0001 C CNN
+	1    6600 3850
+	-1   0    0    -1
+$EndComp
+Wire Wire Line
+	8000 3950 8000 4100
+Wire Wire Line
+	8000 3600 7900 3600
+Connection ~ 8000 3600
+Wire Wire Line
+	8000 3750 8000 3600
+$Comp
+L Device:C_Small C?
+U 1 1 608AC7D8
+P 8000 3850
+AR Path="/608AC7D8" Ref="C?"  Part="1"
+AR Path="/5F9D7A3C/608AC7D8" Ref="C5"  Part="1"
+F 0 "C5" H 8092 3896 50  0000 L CNN
+F 1 "330n" H 8092 3805 50  0000 L CNN
+F 2 "" H 8000 3850 50  0001 C CNN
+F 3 "~" H 8000 3850 50  0001 C CNN
+	1    8000 3850
+	1    0    0    1
+$EndComp
+Wire Wire Line
+	6700 3600 6600 3600
+Wire Wire Line
+	8100 3600 8000 3600
+Text GLabel 8100 3600 2    50   Input ~ 0
+XCVR_VCC
+$Comp
+L custom:L78M05CDT-TR U2
+U 1 1 608A3B2A
+P 7900 3600
+F 0 "U2" H 8500 3865 50  0000 C CNN
+F 1 "L78M05CDT-TR" H 8500 3774 50  0000 C CNN
+F 2 "L78M05CDTTR" H 10450 3850 50  0001 L CNN
+F 3 "https://componentsearchengine.com/Datasheets/2/L78M05CDT-TR.pdf" H 10450 3750 50  0001 L CNN
+F 4 "Linear Voltage Regulators 5.0V 0.5A Positive" H 10450 3650 50  0001 L CNN "Description"
+F 5 "2.4" H 10450 3550 50  0001 L CNN "Height"
+F 6 "511-L78M05CDT-TR" H 10450 3450 50  0001 L CNN "Mouser Part Number"
+F 7 "https://www.mouser.co.uk/ProductDetail/STMicroelectronics/L78M05CDT-TR?qs=JIXmGdi%252BcuKa7ml6d%2FqNIw%3D%3D" H 10450 3350 50  0001 L CNN "Mouser Price/Stock"
+F 8 "STMicroelectronics" H 10450 3250 50  0001 L CNN "Manufacturer_Name"
+F 9 "L78M05CDT-TR" H 10450 3150 50  0001 L CNN "Manufacturer_Part_Number"
+	1    7900 3600
+	-1   0    0    -1
+$EndComp
 Wire Wire Line
 	5750 3600 6600 3600
+$Comp
+L custom:PQS075-S5-S5-S U1
+U 1 1 5FA154A9
+P 3950 3750
+F 0 "U1" H 4100 4050 50  0000 C CNN
+F 1 "PQS075-S5-S5-S" H 3950 3450 50  0000 C CNN
+F 2 "" H 3900 4175 50  0001 C CNN
+F 3 "https://ro.mouser.com/datasheet/2/670/pqs075_s-1893532.pdf" H 3900 4175 50  0001 C CNN
+	1    3950 3750
+	1    0    0    -1
+$EndComp
+$Comp
+L Device:C_Small C?
+U 1 1 5FA20B33
+P 3350 3750
+AR Path="/5FA20B33" Ref="C?"  Part="1"
+AR Path="/5F9D7A3C/5FA20B33" Ref="C2"  Part="1"
+F 0 "C2" H 3250 3700 50  0000 C CNN
+F 1 "4.7u" H 3200 3800 50  0000 C CNN
+F 2 "" H 3350 3750 50  0001 C CNN
+F 3 "~" H 3350 3750 50  0001 C CNN
+	1    3350 3750
+	-1   0    0    1
+$EndComp
+Wire Wire Line
+	3200 3600 3350 3600
+Wire Wire Line
+	4350 3600 4550 3600
+Wire Wire Line
+	4350 3900 4550 3900
+Wire Wire Line
+	2900 3900 3350 3900
+Wire Wire Line
+	3350 3650 3350 3600
+Connection ~ 3350 3600
+Wire Wire Line
+	3350 3600 3550 3600
+Wire Wire Line
+	3350 3850 3350 3900
+Connection ~ 3350 3900
+Wire Wire Line
+	3350 3900 3550 3900
+$Comp
+L Device:C_Small C?
+U 1 1 5FA235C5
+P 4550 3750
+AR Path="/5FA235C5" Ref="C?"  Part="1"
+AR Path="/5F9D7A3C/5FA235C5" Ref="C3"  Part="1"
+F 0 "C3" H 4500 3700 50  0000 C CNN
+F 1 "10u" H 4400 3800 50  0000 C CNN
+F 2 "" H 4550 3750 50  0001 C CNN
+F 3 "~" H 4550 3750 50  0001 C CNN
+	1    4550 3750
+	-1   0    0    1
+$EndComp
+Wire Wire Line
+	4550 3650 4550 3600
+Connection ~ 4550 3600
+Wire Wire Line
+	4550 3600 5550 3600
+Wire Wire Line
+	4550 3850 4550 3900
+Connection ~ 4550 3900
+Wire Wire Line
+	4550 3900 4900 3900
 $EndSCHEMATC

Commit message: Filtering, jumpers, LEDs, misc
* Modified high level diagram to express the shared UART bus
* Renamed XCVR_VCC to XCVR_13V8
* Add solder jumpers on audio, PTT and UART lines for easy prototyping/bypassing
* Added bypass caps on XCVR side data and audio connectors
* Add series ferite beads on data ICs Vcc
* Added schottky diodes to all XCVR_13V8
* Changed series resistors of RXLED/TXLED/VccLED for 6mA current
* Added power LEDs on XCVR_13V8 connector terminals
* Added power LED for XCVR_5V rail
Parts:
- added D1: BG1102W-TR, symbol Device:LED
- added R1: 470, symbol Device:R_Small
Connections:
- net XCVR_5V: now also R1.1
- net XCVR_GND: now also D1.1 (K)
- net XCVR_VCC renamed XCVR_13V8
- new net: D1.2 (A), R1.2
Changed lines of the file:
@@
 	0    -1   -1   0
 $EndComp
-Text GLabel 5650 3250 3    50   Input ~ 0
+Text GLabel 5650 3800 3    50   Input ~ 0
 XCVR_5V
 Text Notes 5800 2800 2    39   ~ 0
@@
 	8100 3600 8000 3600
 Text GLabel 8100 3600 2    50   Input ~ 0
-XCVR_VCC
+XCVR_13V8
 $Comp
 L custom:L78M05CDT-TR U2
@@
 Wire Wire Line
 	4550 3900 4900 3900
+$Comp
+L Device:R_Small R?
+U 1 1 5FDD2952
+P 6000 3850
+AR Path="/5FDD2952" Ref="R?"  Part="1"
+AR Path="/5F9D7A3C/5FDD2952" Ref="R1"  Part="1"
+AR Path="/5F9E7705/5FDD2952" Ref="R?"  Part="1"
+F 0 "R1" H 5900 3850 50  0000 C CNN
+F 1 "470" H 6100 3850 50  0000 C CNN
+F 2 "" H 6000 3850 50  0001 C CNN
+F 3 "~" H 6000 3850 50  0001 C CNN
+	1    6000 3850
+	1    0    0    -1
+$EndComp
+$Comp
+L Device:LED D?
+U 1 1 5FDD2958
+P 6000 4150
+AR Path="/5FDD2958" Ref="D?"  Part="1"
+AR Path="/5F9D7A3C/5FDD2958" Ref="D1"  Part="1"
+AR Path="/5F9E7705/5FDD2958" Ref="D?"  Part="1"
+F 0 "D1" V 6000 4250 50  0000 C CNN
+F 1 "BG1102W-TR" H 5950 4000 50  0000 C CNN
+F 2 "" H 6000 4150 50  0001 C CNN
+F 3 "~" H 6000 4150 50  0001 C CNN
+	1    6000 4150
+	0    -1   -1   0
+$EndComp
+Wire Wire Line
+	6000 3950 6000 4000
+Text GLabel 5950 4450 0    50   Input ~ 0
+XCVR_GND
+Wire Wire Line
+	6000 4450 5950 4450
+Wire Wire Line
+	6000 4300 6000 4450
+Wire Wire Line
+	5650 3250 5650 3700
+Wire Wire Line
+	5650 3700 6000 3700
+Wire Wire Line
+	6000 3700 6000 3750
+Connection ~ 5650 3700
+Wire Wire Line
+	5650 3700 5650 3800
 $EndSCHEMATC

Commit message: Initial footprint placement + changes
* Added initial placement
* Remove pull-down resistors from USB lines.
* Remove ferrite bead from FTDI chip as it was very close to Vcc FB
* Fixed MAX TX pins
* Assigned footprints.
* Removed redundant solder jumpers.
* Small changes for layout coherence.
Parts:
- C1, C2, C3, C4, C5: footprint (none) -> Capacitor_SMD:C_1206_3216Metric_Pad1.42x1.75mm_HandSolder
- D1: footprint (none) -> LED_SMD:LED_1206_3216Metric_Pad1.42x1.75mm_HandSolder
- J1: footprint (none) -> Connector_PinHeader_2.54mm:PinHeader_1x03_P2.54mm_Vertical
- L1: footprint (none) -> Inductor_SMD:L_1206_3216Metric_Pad1.42x1.75mm_HandSolder
- R1: footprint (none) -> Resistor_SMD:R_1206_3216Metric_Pad1.42x1.75mm_HandSolder
- U1: footprint (none) -> custom:SIP-4_PQS075-S5-S5-S
- U2: footprint L78M05CDTTR -> Package_TO_SOT_SMD:TO-252-2
Connections:
- net XCVR_5V: now also D1.2 (A); no longer R1.1
- net XCVR_GND: now also R1.2; no longer D1.1 (K)
- new net: D1.1 (K), R1.1
Other:
- moved on the sheet: D1, R1
Changed lines of the file:
@@
 F 0 "J1" V 5750 3000 50  0000 L CNN
 F 1 "XCVR power choice" V 5850 2700 50  0000 L CNN
-F 2 "" H 5650 3050 50  0001 C CNN
+F 2 "Connector_PinHeader_2.54mm:PinHeader_1x03_P2.54mm_Vertical" H 5650 3050 50  0001 C CNN
 F 3 "~" H 5650 3050 50  0001 C CNN
 	1    5650 3050
@@
 F 0 "L1" V 3050 3600 50  0000 C CNN
 F 1 "6.8u" V 3150 3600 50  0000 C CNN
-F 2 "" H 3100 3600 50  0001 C CNN
+F 2 "Inductor_SMD:L_1206_3216Metric_Pad1.42x1.75mm_HandSolder" H 3100 3600 50  0001 C CNN
 F 3 "~" H 3100 3600 50  0001 C CNN
 	1    3100 3600
@@
 F 0 "C1" H 3000 3700 50  0000 C CNN
 F 1 "4.7u" H 3000 3800 50  0000 C CNN
-F 2 "" H 2900 3750 50  0001 C CNN
+F 2 "Capacitor_SMD:C_1206_3216Metric_Pad1.42x1.75mm_HandSolder" H 2900 3750 50  0001 C CNN
 F 3 "~" H 2900 3750 50  0001 C CNN
 	1    2900 3750
@@
 F 0 "C4" H 6692 3896 50  0000 L CNN
 F 1 "100n" H 6692 3805 50  0000 L CNN
-F 2 "" H 6600 3850 50  0001 C CNN
+F 2 "Capacitor_SMD:C_1206_3216Metric_Pad1.42x1.75mm_HandSolder" H 6600 3850 50  0001 C CNN
 F 3 "~" H 6600 3850 50  0001 C CNN
 	1    6600 3850
@@
 F 0 "C5" H 8092 3896 50  0000 L CNN
 F 1 "330n" H 8092 3805 50  0000 L CNN
-F 2 "" H 8000 3850 50  0001 C CNN
+F 2 "Capacitor_SMD:C_1206_3216Metric_Pad1.42x1.75mm_HandSolder" H 8000 3850 50  0001 C CNN
 F 3 "~" H 8000 3850 50  0001 C CNN
 	1    8000 3850
@@
 F 0 "U2" H 8500 3865 50  0000 C CNN
 F 1 "L78M05CDT-TR" H 8500 3774 50  0000 C CNN
-F 2 "L78M05CDTTR" H 10450 3850 50  0001 L CNN
+F 2 "Package_TO_SOT_SMD:TO-252-2" H 10450 3850 50  0001 L CNN
 F 3 "https://componentsearchengine.com/Datasheets/2/L78M05CDT-TR.pdf" H 10450 3750 50  0001 L CNN
 F 4 "Linear Voltage Regulators 5.0V 0.5A Positive" H 10450 3650 50  0001 L CNN "Description"
@@
 F 0 "U1" H 4100 4050 50  0000 C CNN
 F 1 "PQS075-S5-S5-S" H 3950 3450 50  0000 C CNN
-F 2 "" H 3900 4175 50  0001 C CNN
+F 2 "custom:SIP-4_PQS075-S5-S5-S" H 3900 4175 50  0001 C CNN
 F 3 "https://ro.mouser.com/datasheet/2/670/pqs075_s-1893532.pdf" H 3900 4175 50  0001 C CNN
 	1    3950 3750
@@
 F 0 "C2" H 3250 3700 50  0000 C CNN
 F 1 "4.7u" H 3200 3800 50  0000 C CNN
-F 2 "" H 3350 3750 50  0001 C CNN
+F 2 "Capacitor_SMD:C_1206_3216Metric_Pad1.42x1.75mm_HandSolder" H 3350 3750 50  0001 C CNN
 F 3 "~" H 3350 3750 50  0001 C CNN
 	1    3350 3750
@@
 F 0 "C3" H 4500 3700 50  0000 C CNN
 F 1 "10u" H 4400 3800 50  0000 C CNN
-F 2 "" H 4550 3750 50  0001 C CNN
+F 2 "Capacitor_SMD:C_1206_3216Metric_Pad1.42x1.75mm_HandSolder" H 4550 3750 50  0001 C CNN
 F 3 "~" H 4550 3750 50  0001 C CNN
 	1    4550 3750
@@
 L Device:R_Small R?
 U 1 1 5FDD2952
-P 6000 3850
+P 6000 4200
 AR Path="/5FDD2952" Ref="R?"  Part="1"
 AR Path="/5F9D7A3C/5FDD2952" Ref="R1"  Part="1"
 AR Path="/5F9E7705/5FDD2952" Ref="R?"  Part="1"
-F 0 "R1" H 5900 3850 50  0000 C CNN
-F 1 "470" H 6100 3850 50  0000 C CNN
-F 2 "" H 6000 3850 50  0001 C CNN
-F 3 "~" H 6000 3850 50  0001 C CNN
-	1    6000 3850
+F 0 "R1" H 5900 4200 50  0000 C CNN
+F 1 "470" H 5900 4100 50  0000 C CNN
+F 2 "Resistor_SMD:R_1206_3216Metric_Pad1.42x1.75mm_HandSolder" H 6000 4200 50  0001 C CNN
+F 3 "~" H 6000 4200 50  0001 C CNN
+	1    6000 4200
 	1    0    0    -1
 $EndComp
@@
 L Device:LED D?
 U 1 1 5FDD2958
-P 6000 4150
+P 6000 3900
 AR Path="/5FDD2958" Ref="D?"  Part="1"
 AR Path="/5F9D7A3C/5FDD2958" Ref="D1"  Part="1"
 AR Path="/5F9E7705/5FDD2958" Ref="D?"  Part="1"
-F 0 "D1" V 6000 4250 50  0000 C CNN
-F 1 "BG1102W-TR" H 5950 4000 50  0000 C CNN
-F 2 "" H 6000 4150 50  0001 C CNN
-F 3 "~" H 6000 4150 50  0001 C CNN
-	1    6000 4150
+F 0 "D1" V 6000 4000 50  0000 C CNN
+F 1 "BG1102W-TR" H 6000 3750 50  0000 C CNN
+F 2 "LED_SMD:LED_1206_3216Metric_Pad1.42x1.75mm_HandSolder" H 6000 3900 50  0001 C CNN
+F 3 "~" H 6000 3900 50  0001 C CNN
+	1    6000 3900
 	0    -1   -1   0
 $EndComp
 Wire Wire Line
-	6000 3950 6000 4000
+	6000 4050 6000 4100
 Text GLabel 5950 4450 0    50   Input ~ 0
 XCVR_GND

Commit message: Changed L1 to 0805 due to stock issues
Parts:
- L1: footprint Inductor_SMD:L_1206_3216Metric_Pad1.42x1.75mm_HandSolder -> Inductor_SMD:L_0805_2012Metric_Pad1.15x1.40mm_HandSolder
Changed lines of the file:
@@
 F 0 "L1" V 3050 3600 50  0000 C CNN
 F 1 "6.8u" V 3150 3600 50  0000 C CNN
-F 2 "Inductor_SMD:L_1206_3216Metric_Pad1.42x1.75mm_HandSolder" H 3100 3600 50  0001 C CNN
+F 2 "Inductor_SMD:L_0805_2012Metric_Pad1.15x1.40mm_HandSolder" H 3100 3600 50  0001 C CNN
 F 3 "~" H 3100 3600 50  0001 C CNN
 	1    3100 3600
